File: PCB_layout/TTGO_shield_revD.brd (EAGLE design)
At the start: 120.7 x 101.6 mm, 29 parts

Commit message: reroute RevD
Routing:
- net J-UP: track 45.2 -> 191.4 mm, vias 1 -> 3
- net J-RIGHT: track 67.8 -> 123.0 mm
- net J-LEFT: track 63.6 -> 30.6 mm
- net J-DOWN: track 57.4 -> 32.9 mm, vias 2 -> 1
- net GND: track 279.1 -> 297.9 mm, vias 6 -> 4
- net SCL: track 88.8 -> 76.5 mm
- net SDA: track 92.4 -> 84.2 mm
- net VDD: track 318.7 -> 314.8 mm, vias 1 -> 2
- net J-PRESS: track 47.0 -> 48.4 mm
- net RGBLEDS: track 10.8 -> 9.45 mm
- net CAP2: track 47.0 -> 47.8 mm
