File: PCB_layout/TTGO_shield_revE.sch (EAGLE design)
At the start: 30 parts

Commit message: housekeeping, revE WIP
don't forget to copy over the lbr into the correct location on your computer
Parts:
- removed HEMA1: 10120045-400LF, BadgeParts:10120045-400LF
- added U$1: 10120045-400LF, BadgeParts:10120045-400LF
Connections:
- net GND: no longer HEMA1.D
- net SCL: no longer HEMA1.C
- net SDA: no longer HEMA1.B
- net VDD: no longer HEMA1.A
Other:
- moved on the sheet: MAIN
Changed lines of the file:
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@@
 <part name="GND4" library="SparkFun-PowerSymbols" library_urn="urn:adsk.eagle:library:530" deviceset="GND" device=""/>
 <part name="SUPPLY4" library="SparkFun-PowerSymbols" library_urn="urn:adsk.eagle:library:530" deviceset="5V" device=""/>
-<part name="HEMA1" library="BadgeParts" deviceset="10120045-400LF" device=""/>
-<part name="GND6" library="SparkFun-PowerSymbols" library_urn="urn:adsk.eagle:library:530" deviceset="GND" device=""/>
-<part name="SUPPLY6" library="SparkFun-PowerSymbols" library_urn="urn:adsk.eagle:library:530" deviceset="VDD" device=""/>
 <part name="S1" library="BadgeParts" deviceset="JS1400BFQ" device=""/>
 <part name="GND7" library="SparkFun-PowerSymbols" library_urn="urn:adsk.eagle:library:530" deviceset="GND" device=""/>
@@
 <part name="C9" library="SparkFun-Capacitors" library_urn="urn:adsk.eagle:library:510" deviceset="0.1UF" device="-0603-25V-5%" package3d_urn="urn:adsk.eagle:package:37414/1" value="0.1uF"/>
 <part name="C10" library="SparkFun-Capacitors" library_urn="urn:adsk.eagle:library:510" deviceset="0.1UF" device="-0603-25V-5%" package3d_urn="urn:adsk.eagle:package:37414/1" value="0.1uF"/>
+<part name="U$1" library="BadgeParts" deviceset="10120045-400LF" device=""/>
 </parts>
 <sheets>
@@
 <instance part="GND4" gate="1" x="15.24" y="33.02" rot="R90"/>
 <instance part="SUPPLY4" gate="G$1" x="-35.56" y="2.54" rot="R90"/>
-<instance part="HEMA1" gate="G$1" x="-96.52" y="48.26" rot="R180"/>
-<instance part="GND6" gate="1" x="-86.36" y="33.02"/>
-<instance part="SUPPLY6" gate="VDD" x="-86.36" y="48.26"/>
 <instance part="S1" gate="G$1" x="-12.7" y="-33.02"/>
 <instance part="GND7" gate="1" x="25.4" y="-33.02" rot="R90"/>
@@
 <instance part="C9" gate="G$1" x="53.34" y="-73.66"/>
 <instance part="C10" gate="G$1" x="53.34" y="-93.98"/>
+<instance part="U$1" gate="G$1" x="-7.62" y="76.2"/>
 </instances>
 <busses>
@@
 <pinref part="SUPPLY3" gate="VDD" pin="VDD"/>
 <wire x1="-25.4" y1="48.26" x2="-33.02" y2="48.26" width="0.1524" layer="91"/>
-</segment>
-<segment>
-<pinref part="HEMA1" gate="G$1" pin="A"/>
-<wire x1="-91.44" y1="45.72" x2="-86.36" y2="45.72" width="0.1524" layer="91"/>
-<wire x1="-86.36" y1="45.72" x2="-86.36" y2="48.26" width="0.1524" layer="91"/>
-<pinref part="SUPPLY6" gate="VDD" pin="VDD"/>
 </segment>
 <segment>
@@
 </segment>
 <segment>
-<pinref part="HEMA1" gate="G$1" pin="D"/>
-<pinref part="GND6" gate="1" pin="GND"/>
-<wire x1="-91.44" y1="38.1" x2="-86.36" y2="38.1" width="0.1524" layer="91"/>
-<wire x1="-86.36" y1="38.1" x2="-86.36" y2="35.56" width="0.1524" layer="91"/>
-</segment>
-<segment>
 <pinref part="S1" gate="G$1" pin="5_COM"/>
 <pinref part="GND7" gate="1" pin="GND"/>
@@
 <label x="22.86" y="35.56" size="1.778" layer="95" xref="yes"/>
 </segment>
-<segment>
-<pinref part="HEMA1" gate="G$1" pin="B"/>
-<wire x1="-91.44" y1="43.18" x2="-88.9" y2="43.18" width="0.1524" layer="91"/>
-<label x="-88.9" y="43.18" size="1.778" layer="95" xref="yes"/>
-</segment>
 </net>
 <net name="SCL" class="0">
@@
 <label x="22.86" y="43.18" size="1.778" layer="95" xref="yes"/>
 </segment>
-<segment>
-<pinref part="HEMA1" gate="G$1" pin="C"/>
-<label x="-81.28" y="40.64" size="1.778" layer="95" xref="yes"/>
-<wire x1="-91.44" y1="40.64" x2="-81.28" y2="40.64" width="0.1524" layer="91"/>
-</segment>
-</net>
+</net>

Commit message: RevE off to fab house!
Parts:
- removed U$1: 10120045-400LF, BadgeParts:10120045-400LF
- added C11: 1.0uF, SparkFun-Capacitors:1.0UF-0805-25V-10%
- added CAP1, CAP2: CAPSENSE_BUTTON, BadgeParts:CAPSENSE_BUTTON
- added HEMA1: 10120045-400LF, BadgeParts:10120045-400LF
- added J1, J2, J3, J4, J5: (no value), SparkFun-Connectors:CONN_04LONGPADS
- added LS1: CT-1205H-SMT-TR, BadgeParts:CT-1205H-SMT-TR
- added LTSNS1: LTR-329ALS-01, NickParts:LTR-329ALS-01
- added R1, R2: 4.7k, SparkFun-Resistors:4.7KOHM-0603-1/10W-1%
- added R10: 220, SparkFun-Resistors:470OHM-0603-1/10W-1%
Connections:
- removed net CAP1: MAIN.32
- removed net CAP2: MAIN.33
- new net 15: MAIN.15, R10.1
- new net 25: J3.1, J3.2, J3.3, J3.4, MAIN.25
- new net 26: J4.1, J4.2, J4.3, J4.4, MAIN.26
- new net 27: J5.1, J5.2, J5.3, J5.4, MAIN.27
- new net 32: CAP2.BTN, MAIN.32
- new net 33: CAP1.BTN, MAIN.33
- new net 34: J1.1, J1.2, J1.3, J1.4, MAIN.34
- new net 35: J2.1, J2.2, J2.3, J2.4, MAIN.35
- new net N$7: LS1.1, R10.2
- net GND: now also C11.2, HEMA1.D, LS1.2, LTSNS1.GND
- net SCL: now also HEMA1.C, LTSNS1.SCL, R2.1
- net SDA: now also HEMA1.B, LTSNS1.SDA, R1.1
- net VDD: now also C11.1, HEMA1.A, LTSNS1.VDD, R1.2, R2.2
Other:
- moved on the sheet: R7, R9
