File: PCB_layout/i2c module/module.brd (EAGLE design)
At the start: 38.1 x 38.1 mm, 7 parts, among them IC1 ATTINY85-20SU, J1 M20-9980346

Commit message: reorg, i2c dev, lbr updates
Parts:
- removed JP1, JP2, JP3, JP4: (no value), pinhead:1X04
- added POWER: (no value), SparkFun-LED:LED_3MM
- added R1: 220, SparkFun-Resistors:AXIAL-0.3
- moved IC1 13.7 mm to (6.98, 45.1), turned to 0 degrees
- moved J1 8.23 mm to (26.9, 42.2), turned to 0 degrees
- moved U$1 2.60 mm to (11.4, 3.59)
Connections:
- new net N$11: POWER.A, R1.P$1
- new net PIN0: IC1.PB0
- new net PIN1: IC1.PB1
- new net PIN2: IC1.PB2
- net GND: now also IC1.GND, R1.P$2; no longer IC1.4, JP4.1, JP4.2, JP4.3, JP4.4
- net MISO: no longer IC1.6
- net PIN3: now also IC1.PB3; no longer IC1.2, JP1.1, JP1.2, JP1.3, JP1.4
- net PIN4: now also IC1.PB4; no longer IC1.3, JP2.1, JP2.2, JP2.3, JP2.4
- net RST: now also IC1.PB5; no longer IC1.1
- net SCL: no longer IC1.7
- net SDA: no longer IC1.5
- net VCC: now also IC1.VCC, POWER.K; no longer IC1.8, JP3.1, JP3.2, JP3.3, JP3.4
Routing:
- net VCC: track 81.0 -> 0.00 mm, vias 1 -> 5
- net GND: track 68.1 -> 0.00 mm, vias 1 -> 5
- net SCL: track 49.5 -> 0.00 mm, vias 2 -> 0
- net SDA: track 43.8 -> 0.00 mm, vias 1 -> 0
- net PIN4: track 20.0 -> 0.00 mm, vias 1 -> 5
- net MISO: track 18.5 -> 0.00 mm
- net RST: track 18.0 -> 0.00 mm, vias 0 -> 5
- net PIN3: track 17.7 -> 0.00 mm, vias 1 -> 5
Other:
- board size 38.1 x 38.1 mm -> 100 x 100 mm
- board text added: "0"
- board text added: "1"
- board text added: "2"
- board text added: "3"
- board text added: "4"
- board text added: "5"
- board text added: "< V-Groove"
- board text added: "GND"
- board text added: "VCC"
- board text added: "^ V-Groove"

Commit message: i2c, lbr updates
Parts:
- U$1: value 10120045-400LF -> HEMA-I2C; device BadgeParts:10120045-400LF -> BadgeParts:HEMA-I2C
- moved U$1 4.39 mm to (8.89, 0.00)
Connections:
- removed net MISO: J1.1
- removed net SCL: J1.3, U$1.C
- new net SLC: U$1.B
- net PIN1: now also J1.1
- net PIN2: now also J1.3
- net SDA: now also U$1.C; no longer U$1.D
- net VCC: now also U$1.D; no longer U$1.B

Commit message: PCB design/lib updates
Parts:
- added 0, 1, 2, 3, 4, 5: 3X-PADS-CONNECTED, BadgeParts:3X-PADS
- added GND, VCC: 10X-PADS, BadgeParts:10X-PADS
- added P1: PROTO_VIAS_01X01-1.2, dp_devices:PROTO_VIAS_01X01_1.2
- added POWER1: (no value), SparkFun-LED:LED_3MM
- added R2: 220, SparkFun-Resistors:AXIAL-0.3
- added U$2: 7X-PADS-NC, BadgeParts:7X-PADS-NC
- moved POWER 13.4 mm to (4.09, 42.0), turned to 270 degrees
- moved IC1 11.5 mm to (16.6, 38.8)
- moved J1 10.1 mm to (16.8, 43.2)
- moved R1 8.21 mm to (9.17, 42.6), turned to 270 degrees
Connections:
- removed net PIN0: IC1.PB0
- removed net PIN1: IC1.PB1, J1.1
- removed net PIN2: IC1.PB2, J1.3
- removed net PIN3: IC1.PB3
- removed net PIN4: IC1.PB4
- removed net RST: IC1.PB5, J1.5
- removed net SDA: J1.4, U$1.C
- removed net SLC: U$1.B
- new net N$1: POWER1.A, R2.P$1
- new net N$2: P1.1, R2.P$2
- new net PB0: 0.P$1, 0.P$2, 0.P$3, IC1.PB0, J1.PB0, U$1.C
- new net PB1: IC1.PB1, J1.PB1
- new net PB2: 2.P$1, 2.P$2, 2.P$3, IC1.PB2, J1.PB2, U$1.B
- new net PB3: 3.P$1, 3.P$2, 3.P$3, IC1.PB3
- new net PB4: 4.P$1, 4.P$2, 4.P$3, IC1.PB4
- new net PB5: 1.P$1, 1.P$2, 1.P$3, 5.P$1, 5.P$2, 5.P$3, IC1.PB5, J1.PB5
- net GND: now also GND.P$1, GND.P$10, GND.P$2, GND.P$3, GND.P$4, GND.P$5, GND.P$6, GND.P$7, GND.P$8, GND.P$9, J1.GND, POWER.K, POWER1.K; no longer J1.6, R1.P$2
- net VCC: now also J1.VCC, R1.P$2, VCC.P$1, VCC.P$10, VCC.P$2, VCC.P$3, VCC.P$4, VCC.P$5, VCC.P$6, VCC.P$7, VCC.P$8, VCC.P$9; no longer J1.2, POWER.K
Routing:
- net PB2: track 0.00 -> 92.6 mm, vias 0 -> 1
- net GND: track 0.00 -> 74.4 mm, vias 5 -> 0
- net VCC: track 0.00 -> 68.9 mm, vias 5 -> 0
- net PB0: track 0.00 -> 65.5 mm
- net PB5: track 0.00 -> 61.4 mm, vias 0 -> 1
- net PB4: track 0.00 -> 39.0 mm
- net PB3: track 0.00 -> 30.5 mm
- net PB1: track 0.00 -> 29.1 mm
- net N$11: track 0.00 -> 6.36 mm
- net N$1: track 0.00 -> 5.77 mm, vias 1 -> 0
- net N$2: track 0.00 -> 3.29 mm, vias 1 -> 0
Other:
- outline, holes or cut-outs redrawn
- board text removed: "0"
- board text removed: "1"
- board text removed: "2"
- board text removed: "3"
- board text removed: "4"
- board text removed: "5"
- board text removed: "GND"
- board text removed: "VCC"

Commit message: first i2c dongle iteration panelized
Parts:
- added 10, 11, 12, 13, 14, 15, 16, 17, 18, 19, 20, 21, 22, 23, 24, 25, 26, 27, 28, 29, 30, 31, 32, 33, 34, 35, 6, 7, 8, 9: 3X-PADS-CONNECTED, BadgeParts:3X-PADS
- added GND1, GND2, GND3, GND4, GND5, VCC1, VCC2, VCC3, VCC4, VCC5: 10X-PADS, BadgeParts:10X-PADS
- added IC2, IC3, IC4, IC5, IC6: ATTINY85-20SU, BadgeParts:SOT127P798X216-8N
- added J2, J3, J4, J5, J6: M20-9980346, BadgeParts:HDRV6W64P254_2X3_762X508X868P
- added P2, P3, P4, P5, P6: PROTO_VIAS_01X01-1.2, dp_devices:PROTO_VIAS_01X01_1.2
- added POWER10, POWER11, POWER2, POWER3, POWER4, POWER5, POWER6, POWER7, POWER8, POWER9: (no value), SparkFun-LED:LED_3MM
- added R10, R11, R12, R3, R4, R5, R6, R7, R8, R9: 220, SparkFun-Resistors:AXIAL-0.3
- added U$10, U$12, U$4, U$6, U$8: 7X-PADS-NC, BadgeParts:7X-PADS-NC
- added U$11, U$3, U$5, U$7, U$9: HEMA-I2C, BadgeParts:HEMA-I2C
Connections:
- new net GND1: GND1.P$1, GND1.P$10, GND1.P$2, GND1.P$3, GND1.P$4, GND1.P$5, GND1.P$6, GND1.P$7, GND1.P$8, GND1.P$9, IC2.GND, J2.GND, POWER2.K, POWER3.K, U$3.A
- new net GND2: GND2.P$1, GND2.P$10, GND2.P$2, GND2.P$3, GND2.P$4, GND2.P$5, GND2.P$6, GND2.P$7, GND2.P$8, GND2.P$9, IC3.GND, J3.GND, POWER4.K, POWER5.K, U$5.A
- new net GND3: GND3.P$1, GND3.P$10, GND3.P$2, GND3.P$3, GND3.P$4, GND3.P$5, GND3.P$6, GND3.P$7, GND3.P$8, GND3.P$9, IC4.GND, J4.GND, POWER6.K, POWER7.K, U$7.A
- new net GND4: GND4.P$1, GND4.P$10, GND4.P$2, GND4.P$3, GND4.P$4, GND4.P$5, GND4.P$6, GND4.P$7, GND4.P$8, GND4.P$9, IC5.GND, J5.GND, POWER8.K, POWER9.K, U$9.A
- new net GND5: GND5.P$1, GND5.P$10, GND5.P$2, GND5.P$3, GND5.P$4, GND5.P$5, GND5.P$6, GND5.P$7, GND5.P$8, GND5.P$9, IC6.GND, J6.GND, POWER10.K, POWER11.K, U$11.A
- new net N$10: POWER7.A, R8.P$1
- new net N$12: P4.1, R8.P$2
- new net N$13: POWER8.A, R9.P$1
- new net N$14: POWER9.A, R10.P$1
- new net N$15: P5.1, R10.P$2
- new net N$16: POWER10.A, R11.P$1
- new net N$17: POWER11.A, R12.P$1
- new net N$18: P6.1, R12.P$2
- new net N$3: POWER2.A, R3.P$1
- new net N$4: POWER3.A, R4.P$1
- new net N$5: P2.1, R4.P$2
- new net N$6: POWER4.A, R5.P$1
- new net N$7: POWER5.A, R6.P$1
- new net N$8: P3.1, R6.P$2
- new net N$9: POWER6.A, R7.P$1
- new net PB10: 11.P$1, 11.P$2, 11.P$3, 9.P$1, 9.P$2, 9.P$3, IC2.PB5, J2.PB5
- new net PB11: IC2.PB1, J2.PB1
- new net PB12: 16.P$1, 16.P$2, 16.P$3, IC3.PB0, J3.PB0, U$5.C
- new net PB13: 13.P$1, 13.P$2, 13.P$3, IC3.PB3
- new net PB14: 12.P$1, 12.P$2, 12.P$3, IC3.PB4
- new net PB15: 14.P$1, 14.P$2, 14.P$3, IC3.PB2, J3.PB2, U$5.B
- new net PB16: 15.P$1, 15.P$2, 15.P$3, 17.P$1, 17.P$2, 17.P$3, IC3.PB5, J3.PB5
- new net PB17: IC3.PB1, J3.PB1
- new net PB18: 22.P$1, 22.P$2, 22.P$3, IC4.PB0, J4.PB0, U$7.C
- new net PB19: 19.P$1, 19.P$2, 19.P$3, IC4.PB3
- new net PB20: 18.P$1, 18.P$2, 18.P$3, IC4.PB4
- new net PB21: 20.P$1, 20.P$2, 20.P$3, IC4.PB2, J4.PB2, U$7.B
- new net PB22: 21.P$1, 21.P$2, 21.P$3, 23.P$1, 23.P$2, 23.P$3, IC4.PB5, J4.PB5
- new net PB23: IC4.PB1, J4.PB1
- new net PB24: 28.P$1, 28.P$2, 28.P$3, IC5.PB0, J5.PB0, U$9.C
- new net PB25: 25.P$1, 25.P$2, 25.P$3, IC5.PB3
- new net PB26: 24.P$1, 24.P$2, 24.P$3, IC5.PB4
- new net PB27: 26.P$1, 26.P$2, 26.P$3, IC5.PB2, J5.PB2, U$9.B
- new net PB28: 27.P$1, 27.P$2, 27.P$3, 29.P$1, 29.P$2, 29.P$3, IC5.PB5, J5.PB5
- new net PB29: IC5.PB1, J5.PB1
- new net PB30: 34.P$1, 34.P$2, 34.P$3, IC6.PB0, J6.PB0, U$11.C
- new net PB31: 31.P$1, 31.P$2, 31.P$3, IC6.PB3
- new net PB32: 30.P$1, 30.P$2, 30.P$3, IC6.PB4
- new net PB33: 32.P$1, 32.P$2, 32.P$3, IC6.PB2, J6.PB2, U$11.B
- new net PB34: 33.P$1, 33.P$2, 33.P$3, 35.P$1, 35.P$2, 35.P$3, IC6.PB5, J6.PB5
- new net PB35: IC6.PB1, J6.PB1
- new net PB6: 10.P$1, 10.P$2, 10.P$3, IC2.PB0, J2.PB0, U$3.C
- new net PB7: 7.P$1, 7.P$2, 7.P$3, IC2.PB3
- new net PB8: 6.P$1, 6.P$2, 6.P$3, IC2.PB4
- new net PB9: 8.P$1, 8.P$2, 8.P$3, IC2.PB2, J2.PB2, U$3.B
- new net VCC1: IC2.VCC, J2.VCC, R3.P$2, U$3.D, VCC1.P$1, VCC1.P$10, VCC1.P$2, VCC1.P$3, VCC1.P$4, VCC1.P$5, VCC1.P$6, VCC1.P$7, VCC1.P$8, VCC1.P$9
- new net VCC2: IC3.VCC, J3.VCC, R5.P$2, U$5.D, VCC2.P$1, VCC2.P$10, VCC2.P$2, VCC2.P$3, VCC2.P$4, VCC2.P$5, VCC2.P$6, VCC2.P$7, VCC2.P$8, VCC2.P$9
- new net VCC3: IC4.VCC, J4.VCC, R7.P$2, U$7.D, VCC3.P$1, VCC3.P$10, VCC3.P$2, VCC3.P$3, VCC3.P$4, VCC3.P$5, VCC3.P$6, VCC3.P$7, VCC3.P$8, VCC3.P$9
- new net VCC4: IC5.VCC, J5.VCC, R9.P$2, U$9.D, VCC4.P$1, VCC4.P$10, VCC4.P$2, VCC4.P$3, VCC4.P$4, VCC4.P$5, VCC4.P$6, VCC4.P$7, VCC4.P$8, VCC4.P$9
- new net VCC5: IC6.VCC, J6.VCC, R11.P$2, U$11.D, VCC5.P$1, VCC5.P$10, VCC5.P$2, VCC5.P$3, VCC5.P$4, VCC5.P$5, VCC5.P$6, VCC5.P$7, VCC5.P$8, VCC5.P$9
Routing:
- net GND4: track 0.00 -> 111.2 mm
- net GND5: track 0.00 -> 111.2 mm
- net GND3: track 0.00 -> 111.2 mm
- net PB27: track 0.00 -> 99.9 mm
- net PB21: track 0.00 -> 99.9 mm
- net PB9: track 0.00 -> 92.6 mm, vias 0 -> 1
- net PB15: track 0.00 -> 84.7 mm, vias 0 -> 1
- net GND2: track 0.00 -> 75.3 mm
- net GND1: track 0.00 -> 73.8 mm
- net PB16: track 0.00 -> 71.1 mm, vias 0 -> 1
- net PB10: track 0.00 -> 68.9 mm, vias 0 -> 1
- net VCC2: track 0.00 -> 68.4 mm
- net VCC1: track 0.00 -> 68.4 mm
- net PB28: track 0.00 -> 68.0 mm
- net PB22: track 0.00 -> 68.0 mm
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Other:
- outline, holes or cut-outs redrawn
