File: i2c/PCB/module_RevD.sch (EAGLE design)
At the start: 131 parts, among them IC1 ATTINY85-20SU, J1 M20-9980346

Commit message: Rework of revD boards
Parts:
- removed GND, VCC: 10X-PADS, BadgeParts:10X-PADS
- removed R1, R2: 220, SparkFun-Resistors:RESISTORAXIAL-0.3
- added U$124, U$125, U$128, U$129, U$130, U$131, U$132, U$133, U$134, U$135, U$136, U$137, U$138, U$139, U$140, U$141, U$142, U$143: ONE_PAD, BadgeParts:ONE_PAD
- added U$126, U$127: RESISTOR, BadgeParts:RESISTOR
Connections:
- removed net N$3: HELLO.POS, R2.1
- new net N$2: HELLO.POS, U$127.1
- net GND: now also U$100.P, U$124.P, U$125.P, U$128.P, U$129.P, U$130.P, U$131.P, U$132.P, U$133.P, U$99.P; no longer GND.P$1, GND.P$10, GND.P$2, GND.P$3, GND.P$4, GND.P$5, GND.P$6, GND.P$7, GND.P$8, GND.P$9
- net N$1: now also U$126.1; no longer R1.1
- net PB0: now also U$127.2; no longer R2.2
- net VCC: now also U$126.2, U$134.P, U$135.P, U$136.P, U$137.P, U$138.P, U$139.P, U$140.P, U$141.P, U$142.P, U$143.P; no longer R1.2, VCC.P$1, VCC.P$10, VCC.P$2, VCC.P$3, VCC.P$4, VCC.P$5, VCC.P$6, VCC.P$7, VCC.P$8, VCC.P$9
Other:
- moved on the sheet: U$100, U$99
