File: i2c/PCB/module_RevD_panelized.sch (EAGLE design)
At the start: 786 parts, among them IC1 ATTINY85-20SU, IC2 ATTINY85-20SU, IC3 ATTINY85-20SU, IC4 ATTINY85-20SU, IC5 ATTINY85-20SU, IC6 ATTINY85-20SU, J1 M20-9980346, J2 M20-9980346, J3 M20-9980346, J4 M20-9980346, J5 M20-9980346, J6 M20-9980346

Commit message: Rework of revD boards
Parts:
- removed GND, GND1, GND2, GND3, GND4, GND5, VCC, VCC1, VCC2, VCC3, VCC4, VCC5: 10X-PADS, BadgeParts:10X-PADS
- removed R1, R10, R11, R12, R2, R3, R4, R5, R6, R7, R8, R9: 220, SparkFun-Resistors:RESISTORAXIAL-0.3
- added U$739, U$740, U$741, U$742, U$743, U$744, U$745, U$746, U$747, U$748, U$749, U$750, U$751, U$752, U$753, U$754, U$755, U$756, U$757, U$758, U$759, U$760, U$761, U$762, U$763, U$764, U$765, U$766, U$767, U$768, U$769, U$770, U$771, U$772, U$773, U$774, U$775, U$776, U$777, U$778, U$779, U$780, U$781, U$782, U$783, U$784, U$785, U$790, U$791, U$792, U$793, U$794, U$795, U$796, U$797, U$798, U$799, U$800, U$801, U$802, U$803, U$804, U$805, U$806, U$807, U$808, U$809, U$810, U$811, U$812, U$813, U$814, U$815, U$816, U$817, U$818, U$819, U$820, U$821, U$822, U$823, U$824, U$825, U$826, U$827, U$828, U$829, U$830, U$831, U$832, U$833, U$834, U$835, U$839, U$840, U$841, U$842, U$843, U$844, U$845, U$846, U$847, U$848, U$849, U$850, U$851, U$852, U$853, U$854, U$855, U$856, U$857, U$858: ONE_PAD, BadgeParts:ONE_PAD
- added U$786: GND, BadgeParts:ONE_PAD
- added U$787: VCC, BadgeParts:ONE_PAD
- added U$788: SDA, BadgeParts:ONE_PAD
- added U$789: SCL, BadgeParts:ONE_PAD
- added U$836: DECOUPLING_CAP, BadgeParts:DECOUPLING_CAP
- added U$837, U$838: RESISTOR, BadgeParts:RESISTOR
- U$126, U$127, U$265, U$266, U$408, U$409, U$551, U$552, U$694, U$695: value ONE_PAD -> RESISTOR; device BadgeParts:ONE_PAD -> BadgeParts:RESISTOR
- U$194, U$317, U$440, U$563, U$686: value GND -> ONE_PAD
- U$195, U$318, U$441, U$564, U$687: value VCC -> ONE_PAD
- U$196, U$319, U$442, U$565, U$688: value SDA -> ONE_PAD
- U$197, U$320, U$443, U$566, U$689: value SCL -> ONE_PAD
- U$214, U$357, U$500, U$643: value ONE_PAD -> GND
- U$215, U$358, U$501, U$644: value ONE_PAD -> VCC
- U$216, U$359, U$502, U$645: value ONE_PAD -> SDA
- U$217, U$360, U$503, U$646: value ONE_PAD -> SCL
- U$246, U$369, U$492, U$615, U$738: value DECOUPLING_CAP -> ONE_PAD; device BadgeParts:DECOUPLING_CAP -> BadgeParts:ONE_PAD
- U$264, U$407, U$550, U$693: value ONE_PAD -> DECOUPLING_CAP; device BadgeParts:ONE_PAD -> BadgeParts:DECOUPLING_CAP
Connections:
- net GND: now also U$100.P, U$124.P, U$125.P, U$128.P, U$129.P, U$130.P, U$131.P, U$132.P, U$133.P, U$214.P, U$264.1, U$267.P, U$268.P, U$269.P, U$270.P, U$271.P, U$272.P, U$273.P, U$274.P, U$275.P, U$276.P, U$357.P, U$407.1, U$410.P, U$411.P, U$412.P, U$413.P, U$414.P, U$415.P, U$416.P, U$417.P, U$418.P, U$419.P, U$500.P, U$550.1, U$553.P, U$554.P, U$555.P, U$556.P, U$557.P, U$558.P, U$559.P, U$560.P, U$561.P, U$562.P, U$643.P, U$693.1, U$696.P, U$697.P, U$698.P, U$699.P, U$700.P, U$701.P, U$702.P, U$703.P, U$704.P, U$705.P, U$786.P, U$836.1, U$839.P, U$840.P, U$841.P, U$842.P, U$843.P, U$844.P, U$845.P, U$846.P, U$847.P, U$848.P, U$99.P; no longer GND.P$1, GND.P$10, GND.P$2, GND.P$3, GND.P$4, GND.P$5, GND.P$6, GND.P$7, GND.P$8, GND.P$9, GND1.P$1, GND1.P$10, GND1.P$2, GND1.P$3, GND1.P$4, GND1.P$5, GND1.P$6, GND1.P$7, GND1.P$8, GND1.P$9, GND2.P$1, GND2.P$10, GND2.P$2, GND2.P$3, GND2.P$4, GND2.P$5, GND2.P$6, GND2.P$7, GND2.P$8, GND2.P$9, GND3.P$1, GND3.P$10, GND3.P$2, GND3.P$3, GND3.P$4, GND3.P$5, GND3.P$6, GND3.P$7, GND3.P$8, GND3.P$9, GND4.P$1, GND4.P$10, GND4.P$2, GND4.P$3, GND4.P$4, GND4.P$5, GND4.P$6, GND4.P$7, GND4.P$8, GND4.P$9, GND5.P$1, GND5.P$10, GND5.P$2, GND5.P$3, GND5.P$4, GND5.P$5, GND5.P$6, GND5.P$7, GND5.P$8, GND5.P$9, U$194.P, U$246.1, U$317.P, U$369.1, U$440.P, U$492.1, U$563.P, U$615.1, U$686.P, U$738.1
- net N$1: now also U$126.1; no longer R1.1
- net N$10: now also U$695.1; no longer R10.1
- net N$11: now also U$837.1; no longer R11.1
- net N$12: now also U$838.1; no longer R12.1
- net N$2: now also HELLO.POS, U$127.1; no longer POWER1.POS, R3.1
- net N$3: now also POWER1.POS, U$265.1; no longer HELLO.POS, R2.1
- net N$4: now also U$266.1; no longer R4.1
- net N$5: now also U$408.1; no longer R5.1
- net N$6: now also U$409.1; no longer R6.1
- net N$7: now also U$551.1; no longer R7.1
- net N$8: now also U$552.1; no longer R8.1
- net N$9: now also U$694.1; no longer R9.1
- net PB0: now also U$127.2, U$216.P, U$218.P, U$219.P, U$220.P, U$266.2, U$359.P, U$361.P, U$362.P, U$363.P, U$409.2, U$502.P, U$504.P, U$505.P, U$506.P, U$552.2, U$645.P, U$647.P, U$648.P, U$649.P, U$695.2, U$788.P, U$790.P, U$791.P, U$792.P, U$838.2; no longer R10.2, R12.2, R2.2, R4.2, R6.2, R8.2, U$196.P, U$198.P, U$199.P, U$200.P, U$319.P, U$321.P, U$322.P, U$323.P, U$442.P, U$444.P, U$445.P, U$446.P, U$565.P, U$567.P, U$568.P, U$569.P, U$688.P, U$690.P, U$691.P, U$692.P
- net PB1: now also U$221.P, U$222.P, U$223.P, U$364.P, U$365.P, U$366.P, U$507.P, U$508.P, U$509.P, U$650.P, U$651.P, U$652.P, U$793.P, U$794.P, U$795.P; no longer U$201.P, U$202.P, U$203.P, U$324.P, U$325.P, U$326.P, U$447.P, U$448.P, U$449.P, U$570.P, U$571.P, U$572.P, U$693.P, U$694.P, U$695.P
- net PB2: now also U$217.P, U$224.P, U$225.P, U$226.P, U$360.P, U$367.P, U$368.P, U$369.P, U$503.P, U$510.P, U$511.P, U$512.P, U$646.P, U$653.P, U$654.P, U$655.P, U$789.P, U$796.P, U$797.P, U$798.P; no longer U$197.P, U$204.P, U$205.P, U$206.P, U$320.P, U$327.P, U$328.P, U$329.P, U$443.P, U$450.P, U$451.P, U$452.P, U$566.P, U$573.P, U$574.P, U$575.P, U$689.P, U$696.P, U$697.P, U$698.P
- net PB3: now also U$227.P, U$228.P, U$229.P, U$370.P, U$371.P, U$372.P, U$513.P, U$514.P, U$515.P, U$656.P, U$657.P, U$658.P, U$799.P, U$800.P, U$801.P; no longer U$207.P, U$208.P, U$209.P, U$330.P, U$331.P, U$332.P, U$453.P, U$454.P, U$455.P, U$576.P, U$577.P, U$578.P, U$699.P, U$700.P, U$701.P
- net PB4: now also U$230.P, U$231.P, U$232.P, U$373.P, U$374.P, U$375.P, U$516.P, U$517.P, U$518.P, U$659.P, U$660.P, U$661.P, U$802.P, U$803.P, U$804.P; no longer U$210.P, U$211.P, U$212.P, U$333.P, U$334.P, U$335.P, U$456.P, U$457.P, U$458.P, U$579.P, U$580.P, U$581.P, U$702.P, U$703.P, U$704.P
- net PB5: now also U$233.P, U$234.P, U$235.P, U$376.P, U$377.P, U$378.P, U$519.P, U$520.P, U$521.P, U$662.P, U$663.P, U$664.P, U$805.P, U$806.P, U$807.P; no longer U$213.P, U$214.P, U$215.P, U$336.P, U$337.P, U$338.P, U$459.P, U$460.P, U$461.P, U$582.P, U$583.P, U$584.P, U$705.P, U$706.P, U$707.P
- net VCC: now also U$126.2, U$134.P, U$135.P, U$136.P, U$137.P, U$138.P, U$139.P, U$140.P, U$141.P, U$142.P, U$143.P, U$215.P, U$264.2, U$265.2, U$277.P, U$278.P, U$279.P, U$280.P, U$281.P, U$282.P, U$283.P, U$284.P, U$285.P, U$286.P, U$358.P, U$407.2, U$408.2, U$420.P, U$421.P, U$422.P, U$423.P, U$424.P, U$425.P, U$426.P, U$427.P, U$428.P, U$429.P, U$501.P, U$550.2, U$551.2, U$563.P, U$565.P, U$566.P, U$567.P, U$568.P, U$569.P, U$570.P, U$571.P, U$572.P, U$644.P, U$693.2, U$694.2, U$706.P, U$707.P, U$708.P, U$709.P, U$710.P, U$711.P, U$712.P, U$713.P, U$714.P, U$715.P, U$787.P, U$836.2, U$837.2, U$849.P, U$850.P, U$851.P, U$852.P, U$853.P, U$854.P, U$855.P, U$856.P, U$857.P, U$858.P; no longer R1.2, R11.2, R3.2, R5.2, R7.2, R9.2, U$195.P, U$246.2, U$318.P, U$369.2, U$441.P, U$492.2, U$615.2, U$687.P, U$738.2, VCC.P$1, VCC.P$10, VCC.P$2, VCC.P$3, VCC.P$4, VCC.P$5, VCC.P$6, VCC.P$7, VCC.P$8, VCC.P$9, VCC1.P$1, VCC1.P$10, VCC1.P$2, VCC1.P$3, VCC1.P$4, VCC1.P$5, VCC1.P$6, VCC1.P$7, VCC1.P$8, VCC1.P$9, VCC2.P$1, VCC2.P$10, VCC2.P$2, VCC2.P$3, VCC2.P$4, VCC2.P$5, VCC2.P$6, VCC2.P$7, VCC2.P$8, VCC2.P$9, VCC3.P$1, VCC3.P$10, VCC3.P$2, VCC3.P$3, VCC3.P$4, VCC3.P$5, VCC3.P$6, VCC3.P$7, VCC3.P$8, VCC3.P$9, VCC4.P$1, VCC4.P$10, VCC4.P$2, VCC4.P$3, VCC4.P$4, VCC4.P$5, VCC4.P$6, VCC4.P$7, VCC4.P$8, VCC4.P$9, VCC5.P$1, VCC5.P$10, VCC5.P$2, VCC5.P$3, VCC5.P$4, VCC5.P$5, VCC5.P$6, VCC5.P$7, VCC5.P$8, VCC5.P$9
Other:
- moved on the sheet: HELLO1, HELLO2, HELLO3, HELLO4, HELLO5, POWER1, POWER2, POWER3, POWER4, POWER5, U$100, U$124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
