File: CAA-NMC-2019/CAA-NMC.sch (EAGLE design)
At the start: 20 parts, among them IC1 ATTINY85-20SU, J1 M20-9980346

Commit message: all together now
Parts:
- removed U$71: GND, BadgeParts:ONE_PAD
- removed U$72: SDA, BadgeParts:ONE_PAD
- removed U$73: SCL, BadgeParts:ONE_PAD
- removed U$74: VCC, BadgeParts:ONE_PAD
- added U$4: I2C-PADS, BadgeParts:I2C-PADS
Connections:
- net GND: now also U$4.GND; no longer U$71.P
- net PB0: now also U$4.SDA; no longer U$72.P
- net PB2: now also U$4.SCL; no longer U$73.P
- net VCC: now also U$4.VCC; no longer U$74.P
Changed lines of the file:
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@@
 <part name="POWER" library="BadgeParts" deviceset="LED3MM" device=""/>
 <part name="HELLO" library="BadgeParts" deviceset="LED3MM" device=""/>
-<part name="U$71" library="BadgeParts" deviceset="ONE_PAD" device="" value="GND"/>
-<part name="U$74" library="BadgeParts" deviceset="ONE_PAD" device="" value="VCC"/>
-<part name="U$72" library="BadgeParts" deviceset="ONE_PAD" device="" value="SDA"/>
-<part name="U$73" library="BadgeParts" deviceset="ONE_PAD" device="" value="SCL"/>
 <part name="U$123" library="BadgeParts" deviceset="DECOUPLING_CAP" device=""/>
 <part name="U$126" library="BadgeParts" deviceset="RESISTOR" device=""/>
@@
 <part name="U$2" library="BadgeParts" deviceset="SMT-BATTERY-HOLDER" device=""/>
 <part name="U$3" library="BadgeParts" deviceset="THRU-CR-HOLDER" device=""/>
+<part name="U$4" library="BadgeParts" deviceset="I2C-PADS" device=""/>
 </parts>
 <sheets>
@@
 <attribute name="NAME" x="-159.512" y="59.309" size="1.778" layer="95" font="vector"/>
 </instance>
-<instance part="U$71" gate="G$1" x="-12.7" y="33.02" smashed="yes">
-<attribute name="NAME" x="-13.843" y="34.8742" size="1.778" layer="95"/>
-<attribute name="VALUE" x="-13.843" y="29.718" size="1.778" layer="96"/>
-</instance>
-<instance part="U$74" gate="G$1" x="-25.4" y="33.02" smashed="yes">
-<attribute name="NAME" x="-26.543" y="34.8742" size="1.778" layer="95"/>
-<attribute name="VALUE" x="-26.543" y="29.718" size="1.778" layer="96"/>
-</instance>
-<instance part="U$72" gate="G$1" x="0" y="33.02" smashed="yes">
-<attribute name="NAME" x="-1.143" y="34.8742" size="1.778" layer="95"/>
-<attribute name="VALUE" x="-1.143" y="29.718" size="1.778" layer="96"/>
-</instance>
-<instance part="U$73" gate="G$1" x="15.24" y="33.02" smashed="yes">
-<attribute name="NAME" x="14.097" y="34.8742" size="1.778" layer="95"/>
-<attribute name="VALUE" x="14.097" y="29.718" size="1.778" layer="96"/>
-</instance>
 <instance part="U$123" gate="G$1" x="-147.32" y="91.44" smashed="yes">
 <attribute name="NAME" x="-148.57" y="89.15" size="1.27" layer="95" font="vector" rot="R180" align="center"/>
@@
 <instance part="U$2" gate="G$1" x="-132.08" y="127" smashed="yes"/>
 <instance part="U$3" gate="G$1" x="-132.08" y="106.68" smashed="yes"/>
+<instance part="U$4" gate="G$1" x="-86.36" y="129.54" smashed="yes"/>
 </instances>
 <busses>
@@
 </segment>
 <segment>
-<pinref part="U$72" gate="G$1" pin="P"/>
-<wire x1="2.54" y1="33.02" x2="7.62" y2="33.02" width="0.1524" layer="91"/>
-<wire x1="7.62" y1="33.02" x2="7.62" y2="40.64" width="0.1524" layer="91"/>
-<label x="5.08" y="40.64" size="1.778" layer="95"/>
-</segment>
-<segment>
 <pinref part="U$1" gate="G$1" pin="0"/>
 <wire x1="-68.58" y1="96.52" x2="-86.36" y2="96.52" width="0.1524" layer="91"/>
 <label x="-86.36" y="96.52" size="1.778" layer="95"/>
+</segment>
+<segment>
+<wire x1="-86.36" y1="124.46" x2="-99.06" y2="124.46" width="0.1524" layer="91"/>
+<pinref part="U$4" gate="G$1" pin="SDA"/>
+<label x="-99.06" y="124.46" size="1.778" layer="95"/>
 </segment>
 </net>
@@
 </segment>
 <segment>
-<pinref part="U$74" gate="G$1" pin="P"/>
-<wire x1="-22.86" y1="33.02" x2="-17.78" y2="33.02" width="0.1524" layer="91"/>
-<wire x1="-17.78" y1="33.02" x2="-17.78" y2="40.64" width="0.1524" layer="91"/>
-<label x="-20.32" y="40.64" size="1.778" layer="95"/>
-</segment>
-<segment>
 <pinref part="U$1" gate="G$1" pin="VCC"/>
 <wire x1="-68.58" y1="101.6" x2="-86.36" y2="101.6" width="0.1524" layer="91"/>
@@
 <pinref part="U$145" gate="G$1" pin="5"/>
 <label x="-195.58" y="116.84" size="1.778" layer="95"/>
+</segment>
+<segment>
+<pinref part="U$4" gate="G$1" pin="VCC"/>
+<wire x1="-86.36" y1="129.54" x2="-99.06" y2="129.54" width="0.1524" layer="91"/>
+<label x="-99.06" y="129.54" size="1.778" layer="95"/>
 </segment>
 </net>
@@
 </segment>
 <segment>
-<pinref part="U$71" gate="G$1" pin="P"/>
-<wire x1="-10.16" y1="33.02" x2="-5.08" y2="33.02" width="0.1524" layer="91"/>
-<wire x1="-5.08" y1="33.02" x2="-5.08" y2="40.64" width="0.1524" layer="91"/>
-<label x="-7.62" y="40.64" size="1.778" layer="95"/>
-</segment>
-<segment>
 <pinref part="U$1" gate="G$1" pin="GND"/>
 <wire x1="-68.58" y1="99.06" x2="-86.36" y2="99.06" width="0.1524" layer="91"/>
@@
 <label x="-152.4" y="121.92" size="1.778" layer="95"/>
 </segment>
+<segment>
+<wire x1="-86.36" y1="114.3" x2="-99.06" y2="114.3" width="0.1524" layer="91"/>
+<pinref part="U$4" gate="G$1" pin="GND"/>
+<label x="-99.06" y="114.3" size="1.778" layer="95"/>
+</segment>
 </net>
 <net name="PB2" class="0">
@@
 </segment>
 <segment>
-<pinref part="U$73" gate="G$1" pin="P"/>
-<wire x1="17.78" y1="33.02" x2="22.86" y2="33.02" width="0.1524" layer="91"/>
-<wire x1="22.86" y1="33.02" x2="22.86" y2="40.64" width="0.1524" layer="91"/>
-<label x="20.32" y="40.64" size="1.778" layer="95"/>
-</segment>
-<segment>
 <pinref part="U$1" gate="G$1" pin="2"/>
 <wire x1="-68.58" y1="91.44" x2="-86.36" y2="91.44" width="0.1524" layer="91"/>
 <label x="-86.36" y="91.44" size="1.778" layer="95"/>
 </segment>
-</net>
+<segment>
+<wire x1="-86.36" y1="119.38" x2="-99.06" y2="119.38" width="0.1524" layer="91"/>
+<pinref part="U$4" gate="G$1" pin="SCL"/>
+<label x="-99.06" y="119.38" size="1.778" layer="95"/>
+</segment>
+</net>
