File: CAA-NMC-2019/CAA-NMC-OSH_panelized.sch (EAGLE design)
At the start: 17 parts, among them IC1 ATTINY85-20SU, J1 M20-9980346

Commit message: Finalized file for OSH
Parts:
- added D4, D5, D6, D7, D8, D9: WS2812B, BadgeParts:WS2812B
- added HELLO1, HELLO2, POWER1, POWER2: LED3MM, BadgeParts:LED3MM
- added IC2, IC3: ATTINY85-20SU, BadgeParts:ATTINY85-20SU
- added J2, J3: M20-9980346, BadgeParts:M20-9980346
- added R3, R5: 470, SparkFun-Resistors:470OHM-0603-1/10W-1%
- added R4, R6: 10k, SparkFun-Resistors:10KOHM-0603-1/10W-1%
- added U$10, U$18: SMT-BATTERY-HOLDER, BadgeParts:SMT-BATTERY-HOLDER
- added U$11, U$19: THRU-CR-HOLDER, BadgeParts:THRU-CR-HOLDER
- added U$12, U$20: I2C-PADS, BadgeParts:I2C-PADS
- added U$13, U$5: DECOUPLING_CAP, BadgeParts:DECOUPLING_CAP
- added U$14, U$15, U$6, U$7: RESISTOR, BadgeParts:RESISTOR
- added U$16, U$8: SMT-SWITCH, BadgeParts:SMT-SWITCH
- added U$17, U$9: PROTO, BadgeParts:PROTO
Connections:
- new net N$10: D4.DI, R3.1
- new net N$11: POWER2.POS, U$14.1
- new net N$12: HELLO2.POS, U$15.1
- new net N$13: D7.DO, D8.DI
- new net N$14: D8.DO, D9.DI
- new net N$15: D7.DI, R5.1
- new net N$6: POWER1.POS, U$6.1
- new net N$7: HELLO1.POS, U$7.1
- new net N$8: D4.DO, D5.DI
- new net N$9: D5.DO, D6.DI
- net GND: now also D4.CAP1, D4.GND, D5.CAP1, D5.GND, D6.CAP1, D6.GND, D7.CAP1, D7.GND, D8.CAP1, D8.GND, D9.CAP1, D9.GND, HELLO1.NEG, HELLO2.NEG, IC2.GND, IC3.GND, J2.GND, J3.GND, POWER1.NEG, POWER2.NEG, U$10.GND, U$11.GND, U$12.GND, U$13.1, U$17.GND, U$18.GND, U$19.GND, U$20.GND, U$5.1, U$9.GND
- net PB0: now also IC2.PB0, IC3.PB0, J2.PB0/MOSI/SDA, J3.PB0/MOSI/SDA, U$12.SDA, U$15.2, U$17.0, U$20.SDA, U$7.2, U$9.0
- net PB1: now also IC2.PB1, IC3.PB1, J2.PB1/MISO, J3.PB1/MISO, U$17.1, U$9.1
- net PB2: now also IC2.PB2, IC3.PB2, J2.PB2/SCK/SCL, J3.PB2/SCK/SCL, U$12.SCL, U$17.2, U$20.SCL, U$9.2
- net PB3: now also IC2.PB3, IC3.PB3, U$17.3, U$9.3
- net PB4: now also IC2.PB4, IC3.PB4, R3.2, R4.1, R5.2, R6.1, U$17.4, U$9.4
- net PB5: now also IC2.PB5, IC3.PB5, J2.PB5/RST, J3.PB5/RST, U$17.5, U$9.5
- net VBAT: now also U$10.VBAT, U$11.VBAT, U$16.4, U$18.VBAT, U$19.VBAT, U$8.4
- net VCC: now also D4.CAP2, D4.VCC, D5.CAP2, D5.VCC, D6.CAP2, D6.VCC, D7.CAP2, D7.VCC, D8.CAP2, D8.VCC, D9.CAP2, D9.VCC, IC2.VCC, IC3.VCC, R4.2, R6.2, U$12.VCC, U$13.2, U$14.2, U$16.5, U$17.VCC, U$20.VCC, U$5.2, U$6.2, U$8.5, U$9.VCC
- net VUSB: now also J2.VCC, J3.VCC, U$16.6, U$8.6
