File: CAA-NMC-2019/Pacman/OSH-panels/Pacman2-OSH-panels.sch (EAGLE design)
At the start: 10 parts, among them IC1 ATTINY85-20SU, J2 ICSP-LO-SILK

Commit message: more pacman updates
Parts:
- added D3, D4, D5, D6, D7, D8: WS2812B, BadgeParts:WS2812B
- added DECOUPLER1, DECOUPLER2, DECOUPLER3: .1uf, BadgeParts:0603-CAP
- added IC2, IC3, IC4: ATTINY85-20SU, BadgeParts:ATTINY85-20SU
- added J1, J3, J4: ICSP-LO-SILK, BadgeParts:ICSP-LO-SILK
- added R3, R5, R7: 470, SparkFun-Resistors:470OHM-0603-1/10W-1%
- added R4, R6, R8: 10k, SparkFun-Resistors:10KOHM-0603-1/10W-1%
- added U$1, U$6, U$9: SMT-SWITCH, BadgeParts:SMT-SWITCH
- added U$10, U$4, U$7: SMT-BATTERY-HOLDER, BadgeParts:SMT-BATTERY-HOLDER
- added U$11, U$5, U$8: THRU-CR-HOLDER, BadgeParts:THRU-CR-HOLDER
Connections:
- new net N$1: D3.DO, D4.DI
- new net N$2: D3.DI, R3.1
- new net N$4: D5.DO, D6.DI
- new net N$6: D5.DI, R5.1
- new net N$7: D7.DO, D8.DI
- new net N$8: D7.DI, R7.1
- net GND: now also D3.CAP1, D3.GND, D4.CAP1, D4.GND, D5.CAP1, D5.GND, D6.CAP1, D6.GND, D7.CAP1, D7.GND, D8.CAP1, D8.GND, DECOUPLER1.P$1, DECOUPLER2.P$1, DECOUPLER3.P$1, IC2.GND, IC3.GND, IC4.GND, J1.GND, J3.GND, J4.GND, U$10.GND, U$11.GND, U$4.GND, U$5.GND, U$7.GND, U$8.GND
- net PB0: now also IC2.PB0, IC3.PB0, IC4.PB0, J1.PB0/MOSI/SDA, J3.PB0/MOSI/SDA, J4.PB0/MOSI/SDA
- net PB1: now also IC2.PB1, IC3.PB1, IC4.PB1, J1.PB1/MISO, J3.PB1/MISO, J4.PB1/MISO
- net PB2: now also IC2.PB2, IC3.PB2, IC4.PB2, J1.PB2/SCK/SCL, J3.PB2/SCK/SCL, J4.PB2/SCK/SCL
- net PB3: now also IC2.PB3, IC3.PB3, IC4.PB3
- net PB4: now also IC2.PB4, IC3.PB4, IC4.PB4, R3.2, R4.1, R5.2, R6.1, R7.2, R8.1
- net PB5: now also IC2.PB5, IC3.PB5, IC4.PB5, J1.PB5/RST, J3.PB5/RST, J4.PB5/RST
- net VBAT: now also U$1.4, U$10.VBAT, U$11.VBAT, U$4.VBAT, U$5.VBAT, U$6.4, U$7.VBAT, U$8.VBAT, U$9.4
- net VCC: now also D3.CAP2, D3.VCC, D4.CAP2, D4.VCC, D5.CAP2, D5.VCC, D6.CAP2, D6.VCC, D7.CAP2, D7.VCC, D8.CAP2, D8.VCC, DECOUPLER1.P$2, DECOUPLER2.P$2, DECOUPLER3.P$2, IC2.VCC, IC3.VCC, IC4.VCC, R4.2, R6.2, R8.2, U$1.5, U$6.5, U$9.5
- net VUSB: now also J1.VCC, J3.VCC, J4.VCC, U$1.6, U$6.6, U$9.6
